File: Hardware/Basic/G4_TechWatch-BASIC.sch (EAGLE design)
At the start: 44 parts, among them U2 NRF52832_MODULE_MDBT42

Commit message: End Of Class Schematic
Parts:
- added C2: 1u, LinnesLab-Passives:CAPACITOR0603
- added R8, R9: 10k, LinnesLab-Passives:RESISTOR0603
- added SW1, SW2, SW5: SWITCH.MOM, LinnesLab-Switches:SWITCH.MOM
- added U4: PCF8523, LinnesLab-Clocks:PCF8523
- added XTAL3: 32.7680kHz, LinnesLab-Clocks:CRYSTALECS-.327-12.5-12-C-TR
Connections:
- new net N$16: SW1.1, SW1.2
- new net N$18: SW1.3, SW1.4
- new net N$19: U4.OSCO, XTAL3.1
- new net N$20: U4.OSCI, XTAL3.2
- new net N$22: SW2.1, SW2.2
- new net N$23: SW2.3, SW2.4
- new net N$24: SW5.1, SW5.2
- new net N$25: SW5.3, SW5.4
- new net VBATT: U4.VBAT
- net 3.3V: now also C2.1, R8.2, R9.2, U4.VDD
- net GND: now also C2.2, U4.VSS
- net SCL: now also R8.1, U4.SCL
- net SDA: now also R9.1, U4.SDA
Other:
- note added: "Back-up battery if desired"
- note added: "Buttons"
- note added: "Cortex Debugger/ Programmer"
- note added: "I2C Address = 0x68h"
- note added: "Power Management"
- note added: "RTC"
- note added: "Real-Time Clock"
- note added: "SD Card"
- note added: "nRF52832 Module"

Commit message: Updated Schematics
Connections:
- net N$16 renamed SW1
- net N$22 renamed SW2
- net N$24 renamed SW3
- removed net N$18: SW1.3, SW1.4
- removed net N$23: SW2.3, SW2.4
- removed net N$25: SW5.3, SW5.4
- removed net VBATT: U4.VBAT
- net GND: now also SW1.3, SW1.4, SW2.3, SW2.4, SW5.3, SW5.4, USB2.SHIELD
Other:
- note added: "Digital Outputs CS, OLED RESET, OLED DC, OLED [SPI] [I2C] SD.CS (Optional) Card Detect 1 and 2 Digital Inputs 3x Buttons Charge Status Analog Inputs Battery Monitor Analog Outputs"
- moved on the sheet: C2, C20, C21, C5, C6, CHRG2, D4, D5, J2, LDO2, R11, R12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

Commit message: Schematic Step 1 Done
Parts:
- removed SD2: (no value), LinnesLab-Connectors:MICROSD
- removed USB2: USB.MICRO-BIGGERPADS, LinnesLab-Connectors:USB.MICRO-BIGGERPADS
- added J1: FTDI_DEVICESMD, LinnesLab-Connectors:FTDI_DEVICESMD
Connections:
- removed net CD1: SD2.CARD_DETECT
- removed net CD2: SD2.CARD_DETECT1
- removed net SD.CS: SD2.CS
- removed net USB+: USB2.D+
- removed net USB-: USB2.D-
- net 3.3V: no longer SD2.VDD
- net GND: no longer SD2.GND, SD2.GND1, SD2.VSS, USB2.GND, USB2.SHIELD
- net MISO: no longer SD2.DATA_OUT
- net MOSI: no longer SD2.DATA_IN
- net SCK: no longer SD2.SCLK
- net V_USB: no longer USB2.V+
Other:
- note removed: "Connect MISO, MOSI, and SCK to appropriate pins on microcontroller. Those are SPI pins and are generally prespecified. You have more flexibility with the SD.CS pin."
- note removed: "SD Card"
Changed lines of the file:
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@@
 <part name="R6" library="LinnesLab-Passives" deviceset="RESISTOR" device="0603" package3d_urn="urn:adsk.eagle:package:15661944/2" value="10k"/>
 <part name="R7" library="LinnesLab-Passives" deviceset="RESISTOR" device="0603" package3d_urn="urn:adsk.eagle:package:15661944/2" value="390k"/>
-<part name="SUPPLY7" library="LinnesLab-Symbols" deviceset="3.3V" device=""/>
-<part name="GND22" library="LinnesLab-Symbols" deviceset="GND" device=""/>
-<part name="SD2" library="LinnesLab-Connectors" deviceset="MICROSD" device="" package3d_urn="urn:adsk.eagle:package:17873109/2"/>
 <part name="CHRG2" library="LinnesLab-Power" deviceset="MCP73831" device=""/>
 <part name="LDO2" library="LinnesLab-Power" deviceset="MIC5504" device=""/>
 <part name="D4" library="LinnesLab-DiscreteSemi" deviceset="SCHOTTKY" device="-USC" package3d_urn="urn:adsk.eagle:package:15664784/2"/>
 <part name="D5" library="LinnesLab-DiscreteSemi" deviceset="SCHOTTKY" device="-USC" package3d_urn="urn:adsk.eagle:package:15664784/2"/>
-<part name="USB2" library="LinnesLab-Connectors" deviceset="USB.MICRO" device="-BIGGERPADS"/>
 <part name="J2" library="LinnesLab-Connectors" deviceset="CONN_02" device=""/>
 <part name="C5" library="LinnesLab-Passives" deviceset="CAPACITOR" device="0603" package3d_urn="urn:adsk.eagle:package:15661989/2" value="1u"/>
@@
 <part name="GND2" library="LinnesLab-Symbols" deviceset="GND" device=""/>
 <part name="GND5" library="LinnesLab-Symbols" deviceset="GND" device=""/>
+<part name="J1" library="LinnesLab-Connectors" deviceset="FTDI_DEVICE" device="SMD"/>
 </parts>
 <sheets>
@@
 advanced users only</text>
 <text x="401.32" y="149.86" size="4.318" layer="90" font="vector" ratio="15">OLED</text>
-<text x="261.62" y="-48.26" size="1.778" layer="97">Connect MISO, MOSI, and SCK
-to appropriate pins on
-microcontroller. Those are SPI
-pins and are generally prespecified.
-You have more flexibility with the
-SD.CS pin.</text>
 <text x="408.94" y="-27.94" size="1.27" layer="97">I2C Address = 0x68h</text>
 <text x="363.22" y="-30.48" size="1.27" layer="97">Back-up
@@
 <text x="396.24" y="162.56" size="5.08" layer="97" ratio="15">OLED</text>
 <text x="104.14" y="-10.16" size="5.08" layer="97" ratio="15">Power Management</text>
-<text x="266.7" y="27.94" size="5.08" layer="97" ratio="15">SD Card</text>
 <text x="391.16" y="33.02" size="5.08" layer="97" ratio="15">Buttons</text>
 <text x="386.08" y="-58.42" size="5.08" layer="97" ratio="15">Real-Time Clock</text>
@@
 <attribute name="VALUE" x="392.43" y="79.502" size="1.778" layer="96" rot="R180"/>
 </instance>
-<instance part="SUPPLY7" gate="G$1" x="264.16" y="20.32" smashed="yes">
-<attribute name="VALUE" x="264.16" y="23.114" size="1.778" layer="96" align="bottom-center"/>
-</instance>
-<instance part="GND22" gate="G$1" x="264.16" y="-27.94" smashed="yes">
-<attribute name="VALUE" x="264.16" y="-28.194" size="1.778" layer="96" align="top-center"/>
-</instance>
-<instance part="SD2" gate="G$1" x="284.48" y="-2.54" smashed="yes">
-<attribute name="NAME" x="269.24" y="19.05" size="1.778" layer="95"/>
-<attribute name="VALUE" x="287.02" y="19.05" size="1.778" layer="96"/>
-</instance>
 <instance part="CHRG2" gate="G$1" x="147.32" y="-60.96" smashed="yes">
 <attribute name="NAME" x="139.7" y="-55.372" size="1.778" layer="95"/>
@@
 <attribute name="NAME" x="101.6" y="-56.388" size="1.778" layer="95" font="vector"/>
 <attribute name="VALUE" x="101.6" y="-60.452" size="1.778" layer="96" font="vector" align="top-left"/>
-</instance>
-<instance part="USB2" gate="G$1" x="81.28" y="-63.5" smashed="yes">
-<attribute name="NAME" x="76.2" y="-52.07" size="1.778" layer="95"/>
-<attribute name="VALUE" x="76.2" y="-73.66" size="1.778" layer="96"/>
 </instance>
 <instance part="J2" gate="G$1" x="78.74" y="-27.94" smashed="yes">
@@
 <instance part="GND5" gate="G$1" x="452.12" y="7.62" smashed="yes">
 <attribute name="VALUE" x="452.12" y="7.366" size="1.778" layer="96" align="top-center"/>
+</instance>
+<instance part="J1" gate="G$1" x="76.2" y="-60.96" smashed="yes" rot="MR0">
+<attribute name="NAME" x="76.2" y="-50.8" size="1.778" layer="95" rot="MR0"/>
+<attribute name="VALUE" x="76.2" y="-53.34" size="1.778" layer="96" rot="MR0"/>
 </instance>
 </instances>
@@
 </segment>
 <segment>
-<wire x1="266.7" y1="-15.24" x2="264.16" y2="-15.24" width="0.1524" layer="91"/>
-<pinref part="GND22" gate="G$1" pin="GND"/>
-<wire x1="264.16" y1="-15.24" x2="264.16" y2="-20.32" width="0.1524" layer="91"/>
-<wire x1="264.16" y1="-20.32" x2="264.16" y2="-22.86" width="0.1524" layer="91"/>
-<wire x1="264.16" y1="-22.86" x2="264.16" y2="-25.4" width="0.1524" layer="91"/>
-<wire x1="266.7" y1="-20.32" x2="264.16" y2="-20.32" width="0.1524" layer="91"/>
-<junction x="264.16" y="-20.32"/>
-<wire x1="266.7" y1="-22.86" x2="264.16" y2="-22.86" width="0.1524" layer="91"/>
-<junction x="264.16" y="-22.86"/>
-<pinref part="SD2" gate="G$1" pin="VSS"/>
-<pinref part="SD2" gate="G$1" pin="GND"/>
-<pinref part="SD2" gate="G$1" pin="GND1"/>
-</segment>
-<segment>
 <pinref part="C5" gate="G$1" pin="1"/>
 <pinref part="GND34" gate="G$1" pin="GND"/>
@@
 </segment>
 <segment>
-<pinref part="USB2" gate="G$1" pin="GND"/>
 <wire x1="88.9" y1="-68.58" x2="91.44" y2="-68.58" width="0.1524" layer="91"/>
 <pinref part="GND40" gate="G$1" pin="GND"/>
 <wire x1="91.44" y1="-68.58" x2="91.44" y2="-73.66" width="0.1524" layer="91"/>
-<pinref part="USB2" gate="G$1" pin="SHIELD"/>
 <wire x1="88.9" y1="-55.88" x2="91.44" y2="-55.88" width="0.1524" layer="91"/>
 <wire x1="91.44" y1="-55.88" x2="91.44" y2="-68.58" width="0.1524" layer="91"/>
@@
 </segment>
 <segment>
-<pinref part="SUPPLY7" gate="G$1" pin="3.3V"/>
-<wire x1="264.16" y1="20.32" x2="264.16" y2="-12.7" width="0.1524" layer="91"/>
-<wire x1="264.16" y1="-12.7" x2="266.7" y2="-12.7" width="0.1524" layer="91"/>
-<pinref part="SD2" gate="G$1" pin="VDD"/>
-</segment>
-<segment>
 <pinref part="LDO2" gate="G$1" pin="OUT"/>
 <wire x1="157.48" y1="-25.4" x2="162.56" y2="-25.4" width="0.1524" layer="91"/>
@@
 <wire x1="398.78" y1="96.52" x2="373.38" y2="96.52" width="0.1524" layer="91"/>
 </segment>
-<segment>
-<wire x1="261.62" y1="0" x2="266.7" y2="0" width="0.1524" layer="91"/>
-<label x="261.62" y="0" size="1.27" layer="95" rot="R180" xref="yes"/>
-<pinref part="SD2" gate="G$1" pin="SCLK"/>
-</segment>
 </net>
 <net name="MOSI" class="0">
@@
 <wire x1="398.78" y1="93.98" x2="373.38" y2="93.98" width="0.1524" layer="91"/>
 </segment>
-<segment>
-<wire x1="261.62" y1="2.54" x2="266.7" y2="2.54" width="0.1524" layer="91"/>
-<label x="261.62" y="2.54" size="1.27" layer="95" rot="R180" xref="yes"/>
-<pinref part="SD2" gate="G$1" pin="DATA_IN"/>
-</segment>
 </net>
 <net name="MISO" class="0">
@@
 <pinref part="U2" gate="G$1" pin="P0.14"/>
 <label x="127" y="93.98" size="1.27" layer="95" xref="yes"/>
-</segment>
-<segment>
-<wire x1="261.62" y1="5.08" x2="266.7" y2="5.08" width="0.1524" layer="91"/>
-<label x="261.62" y="5.08" size="1.27" layer="95" rot="R180" xref="yes"/>
-<pinref part="SD2" gate="G$1" pin="DATA_OUT"/>
 </segment>
 </net>
@@
 <pinref part="U3" gate="G$1" pin="/CS"/>
 <wire x1="398.78" y1="109.22" x2="373.38" y2="109.22" width="0.1524" layer="91"/>
-</segment>
-</net>
-<net name="CD2" class="0">
-<segment>
-<wire x1="261.62" y1="12.7" x2="266.7" y2="12.7" width="0.1524" layer="91"/>
-<label x="261.62" y="12.7" size="1.27" layer="95" rot="R180" xref="yes"/>
-<pinref part="SD2" gate="G$1" pin="CARD_DETECT1"/>
-</segment>
-</net>
-<net name="CD1" class="0">
-<segment>
-<wire x1="261.62" y1="15.24" x2="266.7" y2="15.24" width="0.1524" layer="91"/>
-<label x="261.62" y="15.24" size="1.27" layer="95" rot="R180" xref="yes"/>
-<pinref part="SD2" gate="G$1" pin="CARD_DETECT"/>
-</segment>
-</net>
-<net name="SD.CS" class="0">
-<segment>
-<wire x1="261.62" y1="-2.54" x2="266.7" y2="-2.54" width="0.1524" layer="91"/>
-<label x="261.62" y="-2.54" size="1.27" layer="95" rot="R180" xref="yes"/>
-<pinref part="SD2" gate="G$1" pin="CS"/>
 </segment>
 </net>
@@
 <net name="V_USB" class="0">
 <segment>
-<pinref part="USB2" gate="G$1" pin="V+"/>
 <pinref part="D5" gate="G$1" pin="A"/>
 <wire x1="101.6" y1="-58.42" x2="96.52" y2="-58.42" width="0.1524" layer="91"/>
@@
 <net name="USB-" class="0">
 <segment>
-<pinref part="USB2" gate="G$1" pin="D-"/>
 <wire x1="88.9" y1="-60.96" x2="93.98" y2="-60.96" width="0.1524" layer="91"/>
 <label x="93.98" y="-60.96" size="1.27" layer="95" xref="yes"/>
@@
 <net name="USB+" class="0">
 <segment>
-<pinref part="USB2" gate="G$1" pin="D+"/>
 <wire x1="88.9" y1="-63.5" x2="93.98" y2="-63.5" width="0.1524" layer="91"/>
 <label x="93.98" y="-63.5" size="1.27" layer="95" xref="yes"/>

Commit message: End of Class 09/21/2022
Connections:
- removed net BATT: R13.1, R14.2
- new net AIN4/BATT: R13.1, R14.2, U2.P0.28/AIN4
- net CHRG.STAT: now also U2.P0.27
Other:
- note added: "SPECIAL / PORT / PIN ON PACKAGE / GPIO(D_or_A) / Comments SDA / P0.25 / pin2 / D25 SCL / P0.26 / pin3 / D26 none / P0.27 / pin4 / D27 -> Used D27 for CHRG.STAT none / P0.28 / pin5 / D28_or_A4 / (low drive, low frequency IO) -> Used A4 for Battery Measurement none / P0.29 / pin6 / D29_or_A5 / (low drive, low frequency IO) none / P0.30 / pin7 / D30_or_A6 none / P0.31 / pin8 / D31_or_A7 / (used for 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"
- note removed: "SPECIAL / PORT / PIN ON PACKAGE / GPIO(D_or_A) / Comments SDA / P0.25 / pin2 / D25 SCL / P0.26 / pin3 / D26 none / P0.27 / pin4 / D27 none / P0.28 / pin5 / D28_or_A4 / (low drive, low frequency IO) none / P0.29 / pin6 / D29_or_A5 / (low drive, low frequency IO) none / P0.30 / pin7 / D30_or_A6 none / P0.31 / pin8 / D31_or_A7 / (used for battery level monitoring on Adafruit boards)"
Changed lines of the file:
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@@
 SCL / P0.26 / pin3 / D26
 none / P0.27 / pin4 / D27
+-&gt; Used D27 for CHRG.STAT
 none / P0.28 / pin5 / D28_or_A4 / (low drive, low frequency IO)
+-&gt; Used A4 for Battery Measurement
 none / P0.29 / pin6 / D29_or_A5 / (low drive, low frequency IO)
 none / P0.30 / pin7 / D30_or_A6
@@
 <label x="134.62" y="-73.66" size="1.27" layer="95" xref="yes"/>
 </segment>
+<segment>
+<pinref part="U2" gate="G$1" pin="P0.27"/>
+<wire x1="78.74" y1="106.68" x2="76.2" y2="106.68" width="0.1524" layer="91"/>
+<label x="76.2" y="106.68" size="1.778" layer="95" rot="R180" xref="yes"/>
+</segment>
 </net>
 <net name="USB-" class="0">
@@
 <wire x1="88.9" y1="-63.5" x2="93.98" y2="-63.5" width="0.1524" layer="91"/>
 <label x="93.98" y="-63.5" size="1.27" layer="95" xref="yes"/>
-</segment>
-</net>
-<net name="BATT" class="0">
-<segment>
-<pinref part="R13" gate="G$1" pin="1"/>
-<pinref part="R14" gate="G$1" pin="2"/>
-<wire x1="190.5" y1="-48.26" x2="190.5" y2="-43.18" width="0.1524" layer="91"/>
-<label x="190.5" y="-45.72" size="1.27" layer="95" xref="yes"/>
 </segment>
 </net>
@@
 </segment>
 </net>
+<net name="AIN4/BATT" class="0">
+<segment>
+<pinref part="U2" gate="G$1" pin="P0.28/AIN4"/>
+<wire x1="78.74" y1="104.14" x2="76.2" y2="104.14" width="0.1524" layer="91"/>
+<label x="76.2" y="104.14" size="1.778" layer="95" rot="R180" xref="yes"/>
+</segment>
+<segment>
+<pinref part="R13" gate="G$1" pin="1"/>
+<pinref part="R14" gate="G$1" pin="2"/>
+<wire x1="190.5" y1="-48.26" x2="190.5" y2="-43.18" width="0.1524" layer="91"/>
+<label x="190.5" y="-45.72" size="1.27" layer="95" xref="yes"/>
+</segment>
+</net>

Commit message: Commit before leaving class
Connections:
- removed net AIN4/BATT: R13.1, R14.2, U2.P0.28/AIN4
- new net AIN7/BATT: R13.1, R14.2, U2.P0.31/AIN7
- new net D7/SD.CS: U2.P0.07
- net CS.OLED: now also U2.P0.16
- net DC.OLED: now also U2.P0.04/AIN2
- net DTR: now also J1.DTR
- net GND: now also J1.CTS, J1.GND
- net RESET.OLED: now also U2.P0.03/AIN1
- net RXD: now also J1.TXO
- net SW1: now also U2.P0.11
- net SW2: now also U2.P0.15
- net SW3: now also U2.P0.28/AIN4
- net TXD: now also J1.RXI
- net V_USB: now also J1.VCC
Other:
- moved on the sheet: J1
Changed lines of the file:
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@@
 <attribute name="VALUE" x="121.92" y="-73.914" size="1.778" layer="96" align="top-center"/>
 </instance>
-<instance part="GND40" gate="G$1" x="91.44" y="-76.2" smashed="yes">
-<attribute name="VALUE" x="91.44" y="-76.454" size="1.778" layer="96" align="top-center"/>
+<instance part="GND40" gate="G$1" x="81.28" y="-71.12" smashed="yes">
+<attribute name="VALUE" x="81.28" y="-71.374" size="1.778" layer="96" align="top-center"/>
 </instance>
 <instance part="GND41" gate="G$1" x="88.9" y="-33.02" smashed="yes">
@@
 <attribute name="VALUE" x="452.12" y="7.366" size="1.778" layer="96" align="top-center"/>
 </instance>
-<instance part="J1" gate="G$1" x="76.2" y="-60.96" smashed="yes" rot="MR0">
-<attribute name="NAME" x="76.2" y="-50.8" size="1.778" layer="95" rot="MR0"/>
-<attribute name="VALUE" x="76.2" y="-53.34" size="1.778" layer="96" rot="MR0"/>
+<instance part="J1" gate="G$1" x="66.04" y="-55.88" smashed="yes" rot="MR0">
+<attribute name="NAME" x="66.04" y="-45.72" size="1.778" layer="95" rot="MR0"/>
+<attribute name="VALUE" x="66.04" y="-48.26" size="1.778" layer="96" rot="MR0"/>
 </instance>
 </instances>
@@
 </segment>
 <segment>
-<wire x1="88.9" y1="-68.58" x2="91.44" y2="-68.58" width="0.1524" layer="91"/>
-<pinref part="GND40" gate="G$1" pin="GND"/>
-<wire x1="91.44" y1="-68.58" x2="91.44" y2="-73.66" width="0.1524" layer="91"/>
-<wire x1="88.9" y1="-55.88" x2="91.44" y2="-55.88" width="0.1524" layer="91"/>
-<wire x1="91.44" y1="-55.88" x2="91.44" y2="-68.58" width="0.1524" layer="91"/>
-<junction x="91.44" y="-68.58"/>
-</segment>
-<segment>
 <pinref part="J2" gate="G$1" pin="1"/>
 <wire x1="86.36" y1="-27.94" x2="88.9" y2="-27.94" width="0.1524" layer="91"/>
@@
 <junction x="452.12" y="17.78"/>
 <pinref part="GND5" gate="G$1" pin="GND"/>
+</segment>
+<segment>
+<pinref part="J1" gate="G$1" pin="GND"/>
+<pinref part="GND40" gate="G$1" pin="GND"/>
+<wire x1="71.12" y1="-63.5" x2="81.28" y2="-63.5" width="0.1524" layer="91"/>
+<wire x1="81.28" y1="-63.5" x2="81.28" y2="-68.58" width="0.1524" layer="91"/>
+<pinref part="J1" gate="G$1" pin="CTS"/>
+<wire x1="71.12" y1="-60.96" x2="81.28" y2="-60.96" width="0.1524" layer="91"/>
+<wire x1="81.28" y1="-60.96" x2="81.28" y2="-63.5" width="0.1524" layer="91"/>
+<junction x="81.28" y="-63.5"/>
 </segment>
 </net>
@@
 <label x="109.22" y="71.12" size="1.27" layer="95" rot="R270" xref="yes"/>
 </segment>
+<segment>
+<pinref part="J1" gate="G$1" pin="TXO"/>
+<wire x1="71.12" y1="-55.88" x2="73.66" y2="-55.88" width="0.1524" layer="91"/>
+<label x="73.66" y="-55.88" size="1.778" layer="95" xref="yes"/>
+</segment>
 </net>
 <net name="TXD" class="0">
@@
 <label x="104.14" y="71.12" size="1.27" layer="95" rot="R270" xref="yes"/>
 </segment>
+<segment>
+<pinref part="J1" gate="G$1" pin="RXI"/>
+<wire x1="71.12" y1="-53.34" x2="83.82" y2="-53.34" width="0.1524" layer="91"/>
+<label x="83.82" y="-53.34" size="1.778" layer="95" xref="yes"/>
+</segment>
 </net>
 <net name="DTR" class="0">
@@
 <pinref part="C14" gate="G$1" pin="1"/>
 <label x="264.16" y="73.66" size="1.27" layer="95" rot="R180" xref="yes"/>
+</segment>
+<segment>
+<pinref part="J1" gate="G$1" pin="DTR"/>
+<wire x1="71.12" y1="-50.8" x2="73.66" y2="-50.8" width="0.1524" layer="91"/>
+<label x="73.66" y="-50.8" size="1.778" layer="95" xref="yes"/>
 </segment>
 </net>
@@
 <wire x1="398.78" y1="104.14" x2="373.38" y2="104.14" width="0.1524" layer="91"/>
 </segment>
+<segment>
+<pinref part="U2" gate="G$1" pin="P0.04/AIN2"/>
+<wire x1="99.06" y1="73.66" x2="99.06" y2="71.12" width="0.1524" layer="91"/>
+<label x="99.06" y="71.12" size="1.27" layer="95" rot="R270" xref="yes"/>
+</segment>
 </net>
 <net name="RESET.OLED" class="0">
@@
 <pinref part="U3" gate="G$1" pin="/RES"/>
 <wire x1="398.78" y1="106.68" x2="373.38" y2="106.68" width="0.1524" layer="91"/>
+</segment>
+<segment>
+<pinref part="U2" gate="G$1" pin="P0.03/AIN1"/>
+<wire x1="96.52" y1="73.66" x2="96.52" y2="71.12" width="0.1524" layer="91"/>
+<label x="96.52" y="71.12" size="1.27" layer="95" rot="R270" xref="yes"/>
 </segment>
 </net>
@@
 <pinref part="U3" gate="G$1" pin="/CS"/>
 <wire x1="398.78" y1="109.22" x2="373.38" y2="109.22" width="0.1524" layer="91"/>
+</segment>
+<segment>
+<pinref part="U2" gate="G$1" pin="P0.16"/>
+<wire x1="124.46" y1="99.06" x2="127" y2="99.06" width="0.1524" layer="91"/>
+<label x="127" y="99.06" size="1.27" layer="95" xref="yes"/>
 </segment>
 </net>
@@
 <wire x1="101.6" y1="-58.42" x2="96.52" y2="-58.42" width="0.1524" layer="91"/>
 <pinref part="SUPPLY13" gate="G$1" pin="V_USB"/>
-<wire x1="96.52" y1="-58.42" x2="88.9" y2="-58.42" width="0.1524" layer="91"/>
 <wire x1="96.52" y1="-55.88" x2="96.52" y2="-58.42" width="0.1524" layer="91"/>
+<pinref part="J1" gate="G$1" pin="VCC"/>
+<wire x1="71.12" y1="-58.42" x2="96.52" y2="-58.42" width="0.1524" layer="91"/>
 <junction x="96.52" y="-58.42"/>
 </segment>
@@
 <pinref part="U2" gate="G$1" pin="P0.27"/>
 <wire x1="78.74" y1="106.68" x2="76.2" y2="106.68" width="0.1524" layer="91"/>
-<label x="76.2" y="106.68" size="1.778" layer="95" rot="R180" xref="yes"/>
-</segment>
-</net>
-<net name="USB-" class="0">
-<segment>
-<wire x1="88.9" y1="-60.96" x2="93.98" y2="-60.96" width="0.1524" layer="91"/>
-<label x="93.98" y="-60.96" size="1.27" layer="95" xref="yes"/>
-</segment>
-</net>
-<net name="USB+" class="0">
-<segment>
-<wire x1="88.9" y1="-63.5" x2="93.98" y2="-63.5" width="0.1524" layer="91"/>
-<label x="93.98" y="-63.5" size="1.27" layer="95" xref="yes"/>
+<label x="76.2" y="106.68" size="1.27" layer="95" rot="R180" xref="yes"/>
 </segment>
 </net>
@@
 <label x="358.14" y="10.16" size="1.27" layer="95" ratio="15" rot="R180" xref="yes"/>
 </segment>
+<segment>
+<pinref part="U2" gate="G$1" pin="P0.11"/>
+<wire x1="124.46" y1="86.36" x2="127" y2="86.36" width="0.1524" layer="91"/>
+<label x="127" y="86.36" size="1.27" layer="95" xref="yes"/>
+</segment>
 </net>
 <net name="SW2" class="0">
@@
 <label x="391.16" y="10.16" size="1.27" layer="95" ratio="15" rot="R180" xref="yes"/>
 </segment>
+<segment>
+<pinref part="U2" gate="G$1" pin="P0.15"/>
+<wire x1="124.46" y1="96.52" x2="127" y2="96.52" width="0.1524" layer="91"/>
+<label x="127" y="96.52" size="1.27" layer="95" xref="yes"/>
+</segment>
 </net>
 <net name="SW3" class="0">
@@
 <label x="429.26" y="10.16" size="1.27" layer="95" ratio="15" rot="R180" xref="yes"/>
 </segment>
-</net>
-<net name="AIN4/BATT" class="0">
 <segment>
 <pinref part="U2" gate="G$1" pin="P0.28/AIN4"/>
 <wire x1="78.74" y1="104.14" x2="76.2" y2="104.14" width="0.1524" layer="91"/>
-<label x="76.2" y="104.14" size="1.778" layer="95" rot="R180" xref="yes"/>
-</segment>
-<segment>
+<label x="76.2" y="104.14" size="1.27" layer="95" rot="R180" xref="yes"/>
+</segment>
+</net>
+<net name="D7/SD.CS" class="0">
+<segment>
+<pinref part="U2" gate="G$1" pin="P0.07"/>
+<wire x1="106.68" y1="73.66" x2="106.68" y2="71.12" width="0.1524" layer="91"/>
+<label x="106.68" y="71.12" size="1.27" layer="95" rot="R270" xref="yes"/>
+</segment>
+</net>
+<net name="AIN7/BATT" class="0">
+<segment>
+<label x="76.2" y="96.52" size="1.27" layer="95" rot="R180" xref="yes"/>
+<pinref part="U2" gate="G$1" pin="P0.31/AIN7"/>
+<wire x1="76.2" y1="96.52" x2="78.74" y2="96.52" width="0.1524" layer="91"/>
+</segment>
+<segment>
